File: pi_power_board.sch (KiCad schematic (older format))
At the start: 26 parts, among them J1 381camcon, J2 Conn_02x04_Odd_Even, Q1 SSM3K335R, Q2 SSM3K335R, Q3 DMG2305UX-7, U1 LM74610, U2 TPS2400, U3 DMMT5401

Commit message: Add files via upload
Other:
- moved on the sheet: J1

Commit message: Add files via upload
Parts:
- D1: value D5V0L1B2T-7 -> ESDA18-1K
Changed lines of the file:
@@
 P 1900 2600
 F 0 "D1" V 1854 2679 50  0000 L CNN
-F 1 "D5V0L1B2T-7" V 1945 2679 50  0000 L CNN
+F 1 "ESDA18-1K" V 1945 2679 50  0000 L CNN
 F 2 "Diode_SMD:D_SOD-523" H 1900 2600 50  0001 C CNN
 F 3 "~" H 1900 2600 50  0001 C CNN

Commit message: Change header to SMT W/through holes
Parts:
- J2: footprint Connector_PinHeader_2.54mm:PinHeader_2x04_P2.54mm_Vertical -> BG120-08-A-0-N-D:BG120-08-A-0-N-D
Changed lines of the file:
@@
 F 0 "J2" H 5000 5767 50  0000 C CNN
 F 1 "Conn_02x04_Odd_Even" H 5000 5676 50  0000 C CNN
-F 2 "Connector_PinHeader_2.54mm:PinHeader_2x04_P2.54mm_Vertical" H 4950 5450 50  0001 C CNN
+F 2 "BG120-08-A-0-N-D:BG120-08-A-0-N-D" H 4950 5450 50  0001 C CNN
 F 3 "~" H 4950 5450 50  0001 C CNN
 	1    4950 5450
