File: pi_power_board.kicad_pcb (KiCad board)
At the start: 2 copper layers, 33.9 x 27 mm, 26 parts, among them J1 381camcon, J2 Conn_02x04_Odd_Even, Q1 SSM3K335R, Q2 SSM3K335R, Q3 DMG2305UX-7, U1 LM74610, U2 TPS2400, U3 DMMT5401

Commit message: DRC fixes
Parts:
- moved R5 0.10 mm to (84.7, 124.6)
Changed lines of the file:
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@@
   (layers
     (0 F.Cu signal)
-    (31 B.Cu signal hide)
+    (31 B.Cu signal)
     (32 B.Adhes user hide)
     (33 F.Adhes user hide)
@@
   (module BG120-08-A-0-N-D:BG120-08-A-0-N-D locked (layer F.Cu)
     (at 96.25 112.18)
-    (fp_text reference J2 (at 3.55 0.02) (layer B.SilkS)
+    (fp_text reference J2 (at 0.05 -5.68) (layer B.SilkS)
       (effects (font (size 1 1) (thickness 0.15)) (justify mirror))
     )
@@
       (effects (font (size 1 1) (thickness 0.15)) (justify mirror))
     )
-    (fp_line (start -3.81 -5.08) (end 3.81 -5.08) (layer F.CrtYd) (width 0.12))
+    (fp_line (start -3.81 -5.08) (end 3.81 -5.08) (layer B.CrtYd) (width 0.12))
     (fp_line (start -3.81 5.08) (end -3.81 -5.08) (layer B.CrtYd) (width 0.12))
     (fp_line (start 3.81 -5.08) (end 3.81 5.08) (layer B.CrtYd) (width 0.12))
@@
   )
   (module Resistor_SMD:R_0805_2012Metric_Pad1.15x1.40mm_HandSolder (layer F.Cu)
-    (at 84.6 124.6 270)
+    (at 84.7 124.6 270)
     (descr "Resistor SMD 0805 (2012 Metric), square (rectangular) end terminal, IPC_7351 nominal with elongated pad for handsoldering. (Body size source: https://docs.google.com/spreadsheets/d/1BsfQQcO9C6DZCsRaXUlFlo91Tg2WpOkGARC1WS5S8t0/edit?usp=sharing), generated with kicad-footprint-generator")
     (tags "resistor handsolder")
@@
   (segment (start 84.33 102) (end 84.32 102.01) (width 0.508) (layer F.Cu) (net 3))
   (segment (start 86.3 102) (end 84.33 102) (width 0.508) (layer F.Cu) (net 3))
-  (segment (start 87.845 111.01) (end 87.845 109.355) (width 0.381) (layer F.Cu) (net 3))
-  (segment (start 87.845 109.355) (end 88.9 108.3) (width 0.381) (layer F.Cu) (net 3))
-  (segment (start 88.9 103.69) (end 88.17 102.96) (width 0.381) (layer F.Cu) (net 3))
-  (segment (start 88.9 108.3) (end 88.9 103.69) (width 0.381) (layer F.Cu) (net 3))
-  (segment (start 87.845 112.96) (end 88.245 113.36) (width 0.381) (layer F.Cu) (net 3))
-  (segment (start 87.845 111.01) (end 87.845 112.96) (width 0.381) (layer F.Cu) (net 3))
+  (segment (start 87.845 111.01) (end 87.845 109.355) (width 0.508) (layer F.Cu) (net 3))
+  (segment (start 87.845 109.355) (end 88.9 108.3) (width 0.508) (layer F.Cu) (net 3))
+  (segment (start 88.9 103.69) (end 88.17 102.96) (width 0.508) (layer F.Cu) (net 3))
+  (segment (start 88.9 108.3) (end 88.9 103.69) (width 0.508) (layer F.Cu) (net 3))
+  (segment (start 87.845 112.96) (end 88.245 113.36) (width 0.508) (layer F.Cu) (net 3))
+  (segment (start 87.845 111.01) (end 87.845 112.96) (width 0.508) (layer F.Cu) (net 3))
   (via (at 80.6 107.1) (size 0.6) (drill 0.5) (layers F.Cu B.Cu) (net 4))
   (segment (start 80.45 106.95) (end 80.6 107.1) (width 0.381) (layer F.Cu) (net 4))
